File: CAD/V1.0.0/TPS613222A_mini_low_power_boost.kicad_pcb (KiCad board)
At the start: 2 copper layers, 22 x 38 mm, 27 parts, among them K1 HEADER_MALE_1X1, K2 TERMINAL_KF235-5.0-2P, K3 HEADER_MALE_1X1, K4 HEADER_MALE_1X1, K5 TERMINAL_KF235-5.0-2P, K6 HEADER_MALE_1X1, U1 TPS613222A

Commit message: Updating open source files.
Parts:
- moved ? 18.9 mm to (111.5, 113.0)
- moved REF** 16.5 mm to (129.5, 113.8)
- moved ? 14.9 mm to (113.5, 113.0)
Changed lines of the file:
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@@
   )
   (footprint "buzzardLabel" (layer "F.Cu")
-    (at 130.4 113 90)
+    (at 111.5 113 90)
     (attr board_only exclude_from_pos_files exclude_from_bom)
     (fp_text reference "" (at 0 0 90) (layer "F.SilkS")
@@
   )
   (footprint "buzzardLabel" (layer "F.Cu")
-    (at 128.4 113 90)
+    (at 113.5 113 90)
     (attr board_only exclude_from_pos_files exclude_from_bom)
     (fp_text reference "" (at 0 0 90) (layer "F.SilkS")
@@
   )
   (footprint "Soldered Graphics:Logo-Front-SolderedFULL-13mm" (layer "F.Cu")
-    (at 113 113 90)
+    (at 129.5 113.8 90)
     (attr board_only exclude_from_pos_files exclude_from_bom)
     (fp_text reference "REF**" (at 0 -0.5 90 unlocked) (layer "F.SilkS") hide
